File: $OpAmpPassXsistorBenchSupply.sch (KiCad schematic (older format))
At the start: 47 parts

Commit message: working on input filter
Parts:
- removed C? (x2): C_EL, ~, symbol C_EL
- added C?: 1000uF, ~, symbol C_EL
- added C?: 4.7uF, ~, symbol C_MKS2
- added C?: 0.1uF, ~, symbol C_CER
- added L?: 100uH, ~, symbol INDUCTOR
- added R? (x9): 1, ~, symbol R_1W
Connections:
- net GND: now also C?.1, C?.1, C?.1
- net Vin-_raw: no longer CON?.2, CON?.3
- new net: L?.1, R?.2
- new net: C?.2, C?.2, C?.2, L?.2
- new net: R?.1, R?.2 (x6)
- new net: R?.2, R?.2
- new net: R?.1, R?.1
- new net Vee_raw: CON?.2, CON?.3
Other:
- moved on the sheet: C?, D?, L?, R?, U?
