File: OpAmpPassXsistorBenchSupply.kicad_pcb (KiCad board)
At the start: 4 copper layers, 99.7 x 99.7 mm, 70 parts, among them CON1 2.5x5.5mm, CON2 2.1x5.5mm, P1 CONN_1, P2 CONN_1, Q1 2N3904, Q2 2N3904, Q3 TIP120, SW1 SPDT, SW2 SPDT, U1 TL431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

Commit message: revision 1 being sent off to PCB house.
Parts:
- added C14: 0.1uF, CERCAP_2_059A, F.Cu at (191.8, 141.6)
- added C15: 0.1uF, CERCAP_2_059A, F.Cu at (181.0, 154.3)
- added C16: 0.1uF, CERCAP_2_059A, F.Cu at (219.1, 144.8)
- added D1: LED, LED_3MM_069A, F.Cu at (193.7, 194.9)
- added D2: LED, LED_3MM_069A, F.Cu at (200.0, 194.9)
- added FB1: FERRITE_BEAD, FERRITE_AXIAL_06_069A, F.Cu at (187.3, 114.3)
- added FB2: FERRITE_BEAD, FERRITE_AXIAL_06_069A, F.Cu at (127.6, 132.1)
- added FB3: FERRITE_BEAD, FERRITE_AXIAL_06_069A, F.Cu at (187.3, 127.0)
- added FB4: FERRITE_BEAD, FERRITE_AXIAL_06_069A, F.Cu at (159.4, 137.8)
- added G***: OSHW-logo_silkscreen-back_4mm, OSHW-logo_silkscreen-back_4mm, F.Cu at (204.5, 183.5)
- added L2: 100uH, 2A, Toroid_V_06_03_069Bi, F.Cu at (146.1, 145.4)
- added Q4: 2N3904, TO-92_Q_EBC, F.Cu at (174.6, 174.6)
- added Q5: 2N3904, TO-92_Q_EBC, F.Cu at (174.6, 181.6)
- added R33: 1, R_AXIAL_0W25_059Bi, F.Cu at (132.1, 154.9)
- added R34: 1, R_AXIAL_0W25_059Bi, F.Cu at (134.6, 154.9)
- added R35: 220, R_AXIAL_0W25_059Bi, F.Cu at (175.9, 197.5)
- added R36: 220, R_AXIAL_0W25_059Bi, F.Cu at (173.4, 197.5)
- added R37: 1k, R_AXIAL_0W25_059Bi, F.Cu at (193.0, 133.3)
- added R38: 1k, R_AXIAL_0W25_059Bi, F.Cu at (168.9, 184.2)
- C1, C3: footprint ELCAP_10_20_V_059A -> MedCap
- C2, C4, C7, C9: footprint C2 -> BOXCAP_02_03_02_059C
- C6, C8: footprint ELCAP_20_52_V_069Bo -> BigCap
- L1: value 10uH -> 100uH, 100mA
- R5, R6: value 1 -> 0
- U1: footprint TO92-123 -> TO-92_U_059Bo
- moved R13 191.8 mm to (152.4, 129.5), turned to 90 degrees
- moved R15 176.6 mm to (154.9, 129.5), turned to 90 degrees
- moved C9 175.7 mm to (153.7, 135.9), turned to 270 degrees
- moved C7 170.7 mm to (128.3, 170.8), turned to 270 degrees
- moved R16 165.4 mm to (157.5, 118.1)
- moved R28 165.2 mm to (158.8, 181.6)
- moved R1 156.0 mm to (190.5, 111.8), turned to 90 degrees
- moved R27 151.8 mm to (158.8, 179.1)
- moved R21 151.2 mm to (158.8, 163.8)
- moved L1 146.1 mm to (208.9, 105.4), turned to 225 degrees
- moved R31 144.8 mm to (178.4, 164.5)
- moved C2 143.7 mm to (194.9, 104.1), turned to 270 degrees
- moved R19 140.8 mm to (158.8, 158.8)
- moved R24 139.1 mm to (158.8, 171.4)
- moved Q2 133.5 mm to (165.7, 143.8)
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Connections:
- C12 pad 1: GND -> Vcc_reg
- C12 pad 2: Vcc_reg -> GND
- C13 pad 1: GND -> Vcc_reg
- C13 pad 2: Vcc_reg -> GND
- C6 pad 1: N-000004 -> N-0000010
- C7 pad 1: N-000004 -> N-0000010
- Q1 pad 3: N-0000027 (its old number) -> /Base
- Q2 pad 3: N-0000027 (its old number) -> /Base
- Q3 pad 1: N-0000027 (its old number) -> /Base
- Q3 pad 3: Shunt+ -> N-0000015
- R1 pad 1: Vcc_filt -> N-0000017
- R10 pad 1: N-000007 (its old number) -> N-0000036
- R10 pad 2: N-000004 -> N-0000011
- R11 pad 1: N-000006 (its old number) -> N-0000011
- R11 pad 2: N-000004 -> N-0000010
- R12 pad 1: N-000005 (its old number) -> N-0000011
- R12 pad 2: N-000004 -> N-0000010
- R13 pad 2: N-0000011 -> N-0000034
- R14 pad 1: N-0000011 -> N-0000034
- R14 pad 2: N-0000027 (its old number) -> /Base
- R15 pad 2: N-0000010 -> N-0000034
- R16 pad 1: N-0000010 -> N-0000034
- R16 pad 2: N-0000027 (its old number) -> /Base
- R5 pad 1: N-000002 -> VREF
- R5 pad 2: N-000008 -> N-000002
- R6 pad 1: N-000002 -> VREF
- R6 pad 2: N-000007 (its old number) -> N-000008
- R7 pad 1: N-000002 -> N-0000036
- R7 pad 2: N-000006 (its old number) -> N-0000011
- R8 pad 1: N-000002 -> N-0000036
- R8 pad 2: N-000005 (its old number) -> N-0000011
- R9 pad 1: N-000008 -> N-0000036
- R9 pad 2: N-000004 -> N-0000011
- RV2 pad 2: Icontrol -> N-0000032
- RV2 pad 3: VREF -> N-000008
- RV3 pad 2: Vcontrol -> N-0000031
- RV3 pad 3: VREF -> N-000002
- SW1 pad 1: N-000002 -> N-0000016
- SW2 pad 3: N-0000027 (its old number) -> /Base
- U2 pad 3: Vcc_reg -> N-0000014
Routing:
- net Vcc_reg: track 0.00 -> 202.6 mm
- net Shunt-: track 0.00 -> 165.9 mm, vias 0 -> 3
- net VREF: track 0.00 -> 84.9 mm, vias 0 -> 3
- net /Base: track 0.00 -> 82.1 mm, vias 0 -> 3
- net GND: track 0.00 -> 71.8 mm
- net Isense: track 0.00 -> 50.6 mm
- net N-0000022: track 0.00 -> 47.9 mm, vias 0 -> 3
- net Icontrol: track 0.00 -> 45.1 mm
- net N-000005: track 0.00 -> 45.1 mm
- net N-000006: track 0.00 -> 36.7 mm
- net N-0000027: track 0.00 -> 36.1 mm, vias 0 -> 3
- net N-0000024: track 0.00 -> 35.4 mm
- net N-0000035: track 0.00 -> 28.1 mm
- net N-0000026: track 0.00 -> 25.8 mm
- net N-000008: track 1.91 -> 24.8 mm
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- added copper zone on F.Cu, net N-0000010
- added copper zone on F.Cu, net N-0000011
- added copper zone on F.Cu, net N-0000015
- added copper zone on F.Cu, net N-0000016
- added copper zone on F.Cu, net N-0000036
- added copper zone on F.Cu, net N-000009
- added copper zone on F.Cu, net Shunt+
- added copper zone on F.Cu, net Vcc_filt
- removed copper zone on F.Cu, net GND
- removed copper zone on Inner1.Cu, net N-000002
- removed copper zone on Inner2.Cu, net N-000009
Other:
- copper layers 4 -> 2
- board text added: "(v1)"
- board text added: "CC"
- board text added: "CV"
- board text added: "OFF"
- board text added: "ON"
- board text added: "Op Amp / Pass-Transistor Bench Supply"
- board text added: "Output Enable"
- board text added: "Power"
- board text added: "github.com/pepaslabs/OpAmpPassXsistorBenchSupply"
